File: Hardware/StrinX_Controller/NRF24L01.kicad_sch (KiCad schematic)
At the start: 6 parts, among them U3 AMS1117-3.3

Commit message: Add device and footprint
Parts:
- C10, C12: footprint (none) -> Capacitor_SMD:C_0603_1608Metric
- C11: renamed from C13; value 47u -> 100u; footprint (none) -> Capacitor_THT:C_Radial_D8.0mm_H11.5mm_P3.50mm
- C9: renamed from C14; value 47u -> 100u; footprint (none) -> Capacitor_THT:C_Radial_D8.0mm_H11.5mm_P3.50mm
- U3: renamed from U2; value ~ -> NRF24L01
- renumbered U3 to U2

Commit message: Update some device connection and Complete PCB
Parts:
- renumbered C9 to C12, C10 to C13, C11 to C14, C12 to C15
Changed lines of the file:
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@@
 		(dnp no)
 		(fields_autoplaced yes)
-		(property "Reference" "C11"
+		(property "Reference" "C14"
 			(at 105.41 56.8959 0)
 			(effects
@@
 			(project ""
 				(path "/60efaa1b-44bb-4814-90d0-8b9990f45080/7fa7defb-07c2-4a3e-a124-ef53c11d77e5"
-					(reference "C11")
+					(reference "C14")
 					(unit 1)
 				)
@@
 		(on_board yes)
 		(dnp no)
-		(property "Reference" "C12"
+		(property "Reference" "C15"
 			(at 118.11 57.1499 0)
 			(effects
@@
 			(project ""
 				(path "/60efaa1b-44bb-4814-90d0-8b9990f45080/7fa7defb-07c2-4a3e-a124-ef53c11d77e5"
-					(reference "C12")
+					(reference "C15")
 					(unit 1)
 				)
@@
 		(on_board yes)
 		(dnp no)
-		(property "Reference" "C10"
+		(property "Reference" "C13"
 			(at 70.358 57.404 0)
 			(effects
@@
 			(project ""
 				(path "/60efaa1b-44bb-4814-90d0-8b9990f45080/7fa7defb-07c2-4a3e-a124-ef53c11d77e5"
-					(reference "C10")
+					(reference "C13")
 					(unit 1)
 				)
@@
 		(on_board yes)
 		(dnp no)
-		(property "Reference" "C9"
+		(property "Reference" "C12"
 			(at 56.642 56.896 0)
 			(effects
@@
 			(project "StrinX_Controller"
 				(path "/60efaa1b-44bb-4814-90d0-8b9990f45080/7fa7defb-07c2-4a3e-a124-ef53c11d77e5"
-					(reference "C9")
-					(unit 1)
-				)
+					(reference "C12")
+					(unit 1)
+				)
