File: Hardware/Reciever/Reciever.kicad_pcb (KiCad board)
At the start: 2 copper layers, 53 x 43 mm, 49 parts, among them J1 BOOT, J2 USB_C_16p, J3 SWD, J4 I2C, J5 UART, J6 Signal, J7 GND, J8 +5V, U1 STM32F103C8T6, U2 AMS1117-3.3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

Commit message: Fix layout
Connections:
- J8 pad 1: +5V -> VBUS
- J8 pad 2: +5V -> VBUS
- J8 pad 3: +5V -> VBUS
- J8 pad 4: +5V -> VBUS
- J8 pad 5: +5V -> VBUS
- J8 pad 6: +5V -> VBUS
- J8 pad 7: +5V -> VBUS
- J8 pad 8: +5V -> VBUS
Routing:
- net VBUS: track 14.8 -> 119.2 mm, vias 0 -> 1
- net +5V: track 92.6 -> 6.95 mm, vias 1 -> 0
- net GND: track 76.2 -> 58.4 mm
Changed lines of the file:
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@@
 			(layers "*.Cu" "*.Mask")
 			(remove_unused_layers no)
-			(net 6 "+5V")
+			(net 8 "VBUS")
 			(pinfunction "Pin_1")
 			(pintype "passive")
@@
 			(layers "*.Cu" "*.Mask")
 			(remove_unused_layers no)
-			(net 6 "+5V")
+			(net 8 "VBUS")
 			(pinfunction "Pin_2")
 			(pintype "passive")
@@
 			(layers "*.Cu" "*.Mask")
 			(remove_unused_layers no)
-			(net 6 "+5V")
+			(net 8 "VBUS")
 			(pinfunction "Pin_3")
 			(pintype "passive")
@@
 			(layers "*.Cu" "*.Mask")
 			(remove_unused_layers no)
-			(net 6 "+5V")
+			(net 8 "VBUS")
 			(pinfunction "Pin_4")
 			(pintype "passive")
@@
 			(layers "*.Cu" "*.Mask")
 			(remove_unused_layers no)
-			(net 6 "+5V")
+			(net 8 "VBUS")
 			(pinfunction "Pin_5")
 			(pintype "passive")
@@
 			(layers "*.Cu" "*.Mask")
 			(remove_unused_layers no)
-			(net 6 "+5V")
+			(net 8 "VBUS")
 			(pinfunction "Pin_6")
 			(pintype "passive")
@@
 			(layers "*.Cu" "*.Mask")
 			(remove_unused_layers no)
-			(net 6 "+5V")
+			(net 8 "VBUS")
 			(pinfunction "Pin_7")
 			(pintype "passive")
@@
 			(layers "*.Cu" "*.Mask")
 			(remove_unused_layers no)
-			(net 6 "+5V")
+			(net 8 "VBUS")
 			(pinfunction "Pin_8")
 			(pintype "passive")
@@
 				(font
 					(size 0.5 0.5)
+					(thickness 0.15)
 				)
 			)
@@
 	)
 	(segment
-		(start 144.54 79.833455)
-		(end 126.76 79.833455)
-		(width 0.5)
-		(layer "F.Cu")
-		(net 1)
-	)
-	(segment
 		(start 155.36 88.66)
 		(end 155.4 88.7)
@@
 	)
 	(segment
-		(start 151.15 112.583455)
-		(end 153.3 110.433455)
-		(width 0.5)
-		(layer "F.Cu")
-		(net 6)
-	)
-	(segment
-		(start 144.54 82.383455)
-		(end 126.76 82.383455)
-		(width 0.5)
-		(layer "F.Cu")
-		(net 6)
-	)
-	(segment
-		(start 153.3 110.433455)
-		(end 153.3 108.483455)
-		(width 0.5)
-		(layer "F.Cu")
-		(net 6)
-	)
-	(segment
 		(start 155.725 109.583455)
 		(end 154.4 109.583455)
@@
 	)
 	(segment
-		(start 148.05 112.583455)
-		(end 151.15 112.583455)
-		(width 0.5)
-		(layer "F.Cu")
-		(net 6)
-	)
-	(via
-		(at 148.05 112.583455)
-		(size 0.6)
-		(drill 0.3)
-		(layers "F.Cu" "B.Cu")
-		(net 6)
-	)
-	(segment
-		(start 148.05 112.583455)
-		(end 122.1 112.583455)
-		(width 0.5)
-		(layer "B.Cu")
-		(net 6)
-	)
-	(segment
-		(start 120.1 89.043455)
-		(end 126.76 82.383455)
-		(width 0.5)
-		(layer "B.Cu")
-		(net 6)
-	)
-	(segment
-		(start 122.1 112.583455)
-		(end 120.1 110.583455)
-		(width 0.5)
-		(layer "B.Cu")
-		(net 6)
-	)
-	(segment
-		(start 120.1 110.583455)
-		(end 120.1 89.043455)
-		(width 0.5)
-		(layer "B.Cu")
-		(net 6)
-	)
-	(segment
 		(start 136 107.983455)
 		(end 136 108.833455)
@@
 	)
 	(segment
+		(start 157.071 102.762455)
+		(end 157.071 101.4)
+		(width 0.5)
+		(layer "F.Cu")
+		(net 8)
+	)
+	(segment
 		(start 156.346 93.279455)
 		(end 156.75 93.683455)
@@
 	)
 	(segment
-		(start 157.071 102.762455)
+		(start 157.071 101.4)
 		(end 157.071 97.454455)
 		(width 0.5)
@@
 		(net 8)
 	)
+	(via
+		(at 157.071 101.4)
+		(size 0.6)
+		(drill 0.3)
+		(layers "F.Cu" "B.Cu")
+		(net 8)
+	)
+	(segment
+		(start 126.76 82.383455)
+		(end 124.416545 82.383455)
+		(width 0.5)
+		(layer "B.Cu")
+		(net 8)
+	)
+	(segment
+		(start 119.9 86.9)
+		(end 119.9 111.4)
+		(width 0.5)
+		(layer "B.Cu")
+		(net 8)
+	)
+	(segment
+		(start 156.549 101.922)
+		(end 157.071 101.4)
+		(width 0.5)
+		(layer "B.Cu")
+		(net 8)
+	)
+	(segment
+		(start 156.549 115.051)
+		(end 156.549 101.922)
+		(width 0.5)
+		(layer "B.Cu")
+		(net 8)
+	)
+	(segment
+		(start 124.416545 82.383455)
+		(end 119.9 86.9)
+		(width 0.5)
+		(layer "B.Cu")
+		(net 8)
+	)
+	(segment
+		(start 119.9 111.4)
+		(end 125.2 116.7)
+		(width 0.5)
+		(layer "B.Cu")
+		(net 8)
+	)
+	(segment
+		(start 126.76 82.383455)
+		(end 144.54 82.383455)
+		(width 0.5)
+		(layer "B.Cu")
+		(net 8)
+	)
+	(segment
+		(start 154.9 116.7)
+		(end 156.549 115.051)
+		(width 0.5)
+		(layer "B.Cu")
+		(net 8)
+	)
+	(segment
+		(start 125.2 116.7)
+		(end 154.9 116.7)
+		(width 0.5)
+		(layer "B.Cu")
+		(net 8)
+	)
