File: Hardware/Reciever/Reciever.kicad_sch (KiCad schematic)
At the start: 49 parts, among them J1 BOOT, J2 USB_C_16p, J3 SWD, J4 I2C, J5 UART, J6 Signal, J7 GND, J8 +5V, U1 STM32F103C8T6, U2 AMS1117-3.3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

Commit message: Fix layout
Connections:
- net +5V: no longer J8.1 (Pin_1), J8.2 (Pin_2), J8.3 (Pin_3), J8.4 (Pin_4), J8.5 (Pin_5), J8.6 (Pin_6), J8.7 (Pin_7), J8.8 (Pin_8)
- net VBUS: now also J8.1 (Pin_1), J8.2 (Pin_2), J8.3 (Pin_3), J8.4 (Pin_4), J8.5 (Pin_5), J8.6 (Pin_6), J8.7 (Pin_7), J8.8 (Pin_8)
Changed lines of the file:
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@@
 			"ADIAdABpAHAAbAB4AHMAaQBSAG0ASQBGAFkAYgByAEMAQwA4AEUANgBHAGwAUwBSAEoAawB1AEwA"
 			"MQBmAHUAUQBBAEEAQwBBAEEAUwBVAFIAQgBWAEMAVABKAHQAUwBnAEYAVwBFAG0AUwBKAEUAbQBT"
-			"AC8ASwBOAGMASABzAEkAeQBRAG8AQQBoAA=="
+			"AC8ASwBOAGMASABzAEkAeQBRAG8AQQBoAEcAMQBjADMAOQBEAHIAdgBwAHAAcwBxAGgAdwAxAEYA"
+			"cgB6AHEAYgBKAHAAdABmAGYAaQBCAFUAMQBWAFgAdABNAFcANwBqAGsATQBFAFIARQBYAFkAZQBn"
+			"AGsAQgBFAHMAUQAyAEYAUQBGAGwAVgAzAGMAaABSAFgAVABzAFAANgBtAHIAbwBIAGYAWQBiAGcA"
+			"TgBJAGEAZwBBAFQAQgBPAGkAcwBDAHUAYgBJADAAMwBOAFIAUQAvAGUAcQBpAGYAMwBSAG8ASwA4"
+			"AEsAdwBzAHIAcABxADkAMQBHADcAVABUAHYANQBQACsAcQBHAEQARQBhAGYAUgBnAGgAQQBCAFoA"
+			"YQBzAGsASwBKAHoAYwArAHYAYwB0ADkALwBiAC8ATwA3AGIAagBhAFgAbABxAHoAZAB0AG0AZgAz"
+			"AHcASQAwAGMATgBiAEIAawBKAEIAMgBVAEEAbwBIAGUAdgBmAGMAOAAvAHYAKwBVAGIAQgB6ADUA"
+			"MgAzADEALwBmAGYAdQBnAFIAWQBRADIARgBvAGsAdgByADcAMQA5AHcALwBxADYASABUAGsARwBm"
+			"AEoAcABTAFYAUQByAG8AawBwAFUAUABiAGYAbwBxAGoAbQBJAGMAdABZADAAeQBrADQAMQBCAEoA"
+			"egBuADUAMQBVAEgAbABLAEMAQwBDAG4ASgBDAGgARgBGAG4ARgBuAGQAWgBtAHUATABEAE0ANgBR"
+			"AGkAWgBVAE8AUgAzAEgATgBnAEoAWgBKAFUASQBEAHkAbgBWADEAZgByAEwAbwAzAFQAMwBIAGoA"
+			"TwA1AGQAVQA2AEoAZwBCAFUAaQBJADAATQBJADYANgA4AGgAUQBpAFIAVAA3AGoAQgA3AHcAKwBE"
+			"AE4AUAByAFYALwA5AFMAZgArAEcARQBTAG0ARgB6AGUAcwAyAHYAUAAvAG0AUABBAHIATABZAHEA"
+			"UgByAHkALwBIAFIAdwBuAGsAbQA2AHEAdwBxAEwAWQA4AFAATwBpAEMAawBEAEkAQQArAEQAVABW"
+			"AFQAVAB6AG4ANQBtAFIAZABmAGUALwBlAHQAZAArAGQAbQByAFIATABTAHgAZABIAG8AMABTAE8A"
+			"bQBuAC8AdQA5AC8AbgAxAFMAQwBoAHAAawA0AEYASQBBAGgASABNAGcAeAArAGQAWgBIAEgAaQBL"
+			"AEsASwBLAEkALwB5AGsAVQBDAGEAdwBpAGkAaQBpAGkAaQBDACsARwB6AC8AKwBpAGcAZwBuADYA"
+			"NgBOAEcAagByADcAdgB1AHUAbgBQAFAAUABiAGUANQB1AGYAbgBPAE8AKwA5AHMAYQBXAGsASgB3"
+			"ADMARABMAGwAaQAzAFAAUABQAFAATQA5AA=="
 		)
 	)
@@
 	)
 	(symbol
+		(lib_id "power:VBUS")
+		(at 361.95 88.9 0)
+		(unit 1)
+		(exclude_from_sim no)
+		(in_bom yes)
+		(on_board yes)
+		(dnp no)
+		(fields_autoplaced yes)
+		(property "Reference" "#PWR027"
+			(at 361.95 92.71 0)
+			(effects
+				(font
+					(size 1.27 1.27)
+				)
+				(hide yes)
+			)
+		)
+		(property "Value" "VBUS"
+			(at 361.95 83.82 0)
+			(effects
+				(font
+					(size 1.27 1.27)
+				)
+			)
+		)
+		(property "Footprint" ""
+			(at 361.95 88.9 0)
+			(effects
+				(font
+					(size 1.27 1.27)
+				)
+				(hide yes)
+			)
+		)
+		(property "Datasheet" ""
+			(at 361.95 88.9 0)
+			(effects
+				(font
+					(size 1.27 1.27)
+				)
+				(hide yes)
+			)
+		)
+		(property "Description" "Power symbol creates a global label with name \"VBUS\""
+			(at 361.95 88.9 0)
+			(effects
+				(font
+					(size 1.27 1.27)
+				)
+				(hide yes)
+			)
+		)
+		(pin "1"
+		)
+		(instances
+			(project "Reciever"
+				(path "/92243f9b-a032-4350-b0ea-04fa935ca57b"
+					(reference "#PWR027")
+					(unit 1)
+				)
+			)
+		)
+	)
+	(symbol
 		(lib_id "Device:C")
 		(at 284.48 31.75 0)
@@
 					(unit 1)
 				)
-			)
-		)
-	)
-	(symbol
-		(lib_id "power:+5V")
-		(at 361.95 88.9 0)
-		(unit 1)
-		(exclude_from_sim no)
-		(in_bom yes)
-		(on_board yes)
-		(dnp no)
-		(fields_autoplaced yes)
-		(property "Reference" "#PWR020"
-			(at 361.95 92.71 0)
-			(effects
-				(font
-					(size 1.27 1.27)
-				)
-				(hide yes)
-			)
-		)
-		(property "Value" "+5V"
-			(at 361.95 83.82 0)
-			(effects
-				(font
-					(size 1.27 1.27)
-				)
-			)
-		)
-		(property "Footprint" ""
-			(at 361.95 88.9 0)
-			(effects
-				(font
-					(size 1.27 1.27)
-				)
-				(hide yes)
-			)
-		)
-		(property "Datasheet" ""
-			(at 361.95 88.9 0)
-			(effects
-				(font
-					(size 1.27 1.27)
-				)
-				(hide yes)
-			)
-		)
-		(property "Description" "Power symbol creates a global label with name \"+5V\""
-			(at 361.95 88.9 0)
-			(effects
-				(font
-					(size 1.27 1.27)
-				)
-				(hide yes)
-			)
-		)
-		(pin "1"
-		)
-		(instances
-			(project "Reciever"
-				(path "/92243f9b-a032-4350-b0ea-04fa935ca57b"
-					(reference "#PWR020")
-					(unit 1)
-				)
